Commit message: Update cognitive_rover.urdf

File: cognitive_rover.urdf (robot description, URDF)
Before this commit: robot cognitive_rover_arm, 6 links, 5 joints
Links:
- removed link arm_base_link
- removed link base_chassis
- removed link elbow_link
- removed link gripper_link
- removed link shoulder_link
- removed link wrist_link
- added link battery; visual box size=0.11 0.04 0.025
- added link caster_wheel; visual sphere radius=0.015
- added link esp32; visual box size=0.052 0.028 0.01
- added link left_wheel; visual cylinder length=0.026 radius=0.0325
- added link lower_deck; visual box size=0.26 0.18 0.01
- added link pca9685; visual box size=0.062 0.025 0.01
- added link pi_camera; visual box size=0.01 0.025 0.025
- added link raspberry_pi; visual box size=0.085 0.056 0.015
- added link right_wheel; visual cylinder length=0.026 radius=0.0325
- added link ultrasonic; visual box size=0.01 0.045 0.02
- added link upper_deck; visual box size=0.26 0.18 0.005
Joints:
- removed joint ch0_base_swivel
- removed joint ch1_shoulder
- removed joint ch2_elbow
- removed joint ch3_wrist
- removed joint ch4_gripper
- added joint battery_joint: type fixed, parent lower_deck, child battery, origin xyz=-0.02 0 0.015 rpy=0 0 0
- added joint camera_joint: type fixed, parent upper_deck, child pi_camera, origin xyz=0.12 0 0.025 rpy=0 0.261 0
- added joint caster_joint: type fixed, parent lower_deck, child caster_wheel, origin xyz=0.10 0 -0.015 rpy=0 0 0
- added joint deck_spacer: type fixed, parent lower_deck, child upper_deck, origin xyz=0 0 0.04 rpy=0 0 0
- added joint esp_joint: type fixed, parent upper_deck, child esp32, origin xyz=-0.08 0.04 0.01 rpy=0 0 0
- added joint left_wheel_joint: type continuous, parent lower_deck, child left_wheel, origin xyz=-0.05 0.105 0 rpy=1.5708 0 0, axis 0 0 1
- added joint pca_joint: type fixed, parent upper_deck, child pca9685, origin xyz=0.02 0 0.01 rpy=0 0 0
- added joint right_wheel_joint: type continuous, parent lower_deck, child right_wheel, origin xyz=-0.05 -0.105 0 rpy=1.5708 0 0, axis 0 0 1
- added joint rpi_joint: type fixed, parent upper_deck, child raspberry_pi, origin xyz=-0.06 -0.045 0.01 rpy=0 0 0
- added joint sonar_joint: type fixed, parent lower_deck, child ultrasonic, origin xyz=0.13 0 0.02 rpy=0 0 0

Commit message: Update cognitive_rover.urdf

File: cognitive_rover.urdf (robot description, URDF)
Before this commit: robot cyberpunk_base, 11 links, 10 joints
Links:
- removed link battery
- removed link caster_wheel
- removed link esp32
- removed link left_wheel
- removed link lower_deck
- removed link pca9685
- removed link pi_camera
- removed link right_wheel
- removed link ultrasonic
- removed link upper_deck
- added link arm_mount_pad; visual cylinder length=0.005 radius=0.04
- added link base_chassis; visual box size=0.28 0.20 0.006
- added link battery_pack; visual box size=0.10 0.035 0.025
- added link fl_wheel; visual cylinder length=0.026 radius=0.0325
- added link fr_wheel; visual cylinder length=0.026 radius=0.0325
- added link microcontroller_cluster; visual box size=0.06 0.05 0.01
- added link motor_driver_left; visual box size=0.045 0.045 0.02
- added link motor_driver_right; visual box size=0.045 0.045 0.02
- added link rear_ui_panel; visual box size=0.01 0.08 0.01
- added link rl_wheel; visual cylinder length=0.026 radius=0.0325
- added link rr_wheel; visual cylinder length=0.026 radius=0.0325
- added link sensor_array; visual box size=0.01 0.06 0.03
Joints:
- removed joint camera_joint
- removed joint caster_joint
- removed joint deck_spacer
- removed joint esp_joint
- removed joint left_wheel_joint
- removed joint pca_joint
- removed joint right_wheel_joint
- removed joint sonar_joint
- added joint arm_mount_joint: type fixed, parent base_chassis, child arm_mount_pad, origin xyz=0.09 0 0.005 rpy=0 0 0
- added joint driver1_joint: type fixed, parent base_chassis, child motor_driver_left, origin xyz=0 0.07 0.015 rpy=0 0 0
- added joint driver2_joint: type fixed, parent base_chassis, child motor_driver_right, origin xyz=0 -0.07 0.015 rpy=0 0 0
- added joint esp_pca_joint: type fixed, parent base_chassis, child microcontroller_cluster, origin xyz=-0.10 -0.06 0.01 rpy=0 0 0
- added joint fl_wheel_joint: type continuous, parent base_chassis, child fl_wheel, origin xyz=0.09 0.115 -0.015 rpy=1.5708 0 0, axis 0 0 1
- added joint fr_wheel_joint: type continuous, parent base_chassis, child fr_wheel, origin xyz=0.09 -0.115 -0.015 rpy=1.5708 0 0, axis 0 0 1
- added joint rl_wheel_joint: type continuous, parent base_chassis, child rl_wheel, origin xyz=-0.09 0.115 -0.015 rpy=1.5708 0 0, axis 0 0 1
- added joint rr_wheel_joint: type continuous, parent base_chassis, child rr_wheel, origin xyz=-0.09 -0.115 -0.015 rpy=1.5708 0 0, axis 0 0 1
- added joint sensor_bracket_joint: type fixed, parent base_chassis, child sensor_array, origin xyz=0.14 0 0.01 rpy=0 0 0
- added joint ui_panel_joint: type fixed, parent base_chassis, child rear_ui_panel, origin xyz=-0.14 0 0.005 rpy=0 0 0
- joint battery_joint: child battery -> battery_pack; parent lower_deck -> base_chassis
- joint rpi_joint: origin xyz=-0.06 -0.045 0.01 rpy=0 0 0 -> xyz=-0.10 0.06 0.01 rpy=0 0 0; parent upper_deck -> base_chassis
